File: mcu.sch (KiCad schematic (older format))
At the start: 15 parts, among them J401 Pwr, U401 MAX485E, U402 LM7812_TO220, U403 74HC595

Commit message: update
Parts:
- A401: symbol MCU_Module:Arduino_Nano_v3.x -> umi6r2-rescue:Arduino_Nano_v3.x-MCU_Module
- C401, C406: symbol Device:CP_Small -> umi6r2-rescue:CP_Small-Device
Changed lines of the file:
@@
 EESchema Schematic File Version 4
-LIBS:umi6r2-cache
 EELAYER 30 0
 EELAYER END
@@
 $EndComp
 $Comp
-L MCU_Module:Arduino_Nano_v3.x A401
+L umi6r2-rescue:Arduino_Nano_v3.x-MCU_Module A401
 U 1 1 5DC741DC
 P 7850 4000
@@
 $EndComp
 $Comp
-L Device:CP_Small C401
+L umi6r2-rescue:CP_Small-Device C401
 U 1 1 5DE25965
 P 4150 1750
+AR Path="/5DE25965" Ref="C401"  Part="1"
+AR Path="/5DB9CE60/5DE25965" Ref="C401"  Part="1"
 F 0 "C401" H 4238 1796 50  0000 L CNN
 F 1 "47u/35V" H 4238 1705 50  0000 L CNN
@@
 $EndComp
 $Comp
-L Device:CP_Small C406
+L umi6r2-rescue:CP_Small-Device C406
 U 1 1 5DE2610A
 P 5950 1750
+AR Path="/5DE2610A" Ref="C406"  Part="1"
+AR Path="/5DB9CE60/5DE2610A" Ref="C406"  Part="1"
 F 0 "C406" H 6038 1796 50  0000 L CNN
 F 1 "100u/16V" H 6038 1705 50  0000 L CNN
