File: relay.sch (KiCad schematic (older format))
At the start: 15 parts, among them J301 OUTPUTS, K301 LEG-12, K302 LEG-12, Q301 BC847, Q302 BC847

Commit message: update
Parts:
- C301, C302: symbol Device:CP_Small -> umi6r2-rescue:CP_Small-Device
Changed lines of the file:
@@
 EESchema Schematic File Version 4
-LIBS:umi6r2-cache
 EELAYER 30 0
 EELAYER END
@@
 	4900 2650 4900 2800
 $Comp
-L Device:CP_Small C301
+L umi6r2-rescue:CP_Small-Device C301
 U 1 1 5DBD1703
 P 4650 2950
+AR Path="/5DBD1703" Ref="C301"  Part="1"
+AR Path="/5DB9CE03/5DBD1703" Ref="C301"  Part="1"
 F 0 "C301" H 4350 2950 50  0000 L CNN
 F 1 "100u/16V" H 4250 2850 50  0000 L CNN
@@
 $EndComp
 $Comp
-L Device:CP_Small C302
+L umi6r2-rescue:CP_Small-Device C302
 U 1 1 5DBD2456
 P 4650 4500
+AR Path="/5DBD2456" Ref="C302"  Part="1"
+AR Path="/5DB9CE03/5DBD2456" Ref="C302"  Part="1"
 F 0 "C302" H 4400 4550 50  0000 L CNN
 F 1 "100u/16V" H 4250 4400 50  0000 L CNN
